File: source/kicad/Krtkus2/Krtkus2.kicad_sch (KiCad schematic)
At the start: 254 parts, among them Q1 Q_NMOS, SW1 SW_Push, SW10 SW_Push, SW11 SW_Push, SW12 SW_Push, SW13 SW_Push, SW14 SW_Push, SW15 SW_Push, SW16 SW_Push, SW17 SW_Push, SW18 SW_Push, SW19 SW_Push, SW2 SW_Push, SW20 SW_Push, SW21 SW_Push, SW22 SW_Push, SW23 SW_Push, SW24 SW_Push, SW25 SW_Push, SW26 SW_Push, SW27 SW_Push, SW28 SW_Push, SW29 SW_Push, SW3 SW_Push, SW30 SW_Push, SW31 SW_Push, SW32 SW_Push, SW33 SW_Push, SW34 SW_Push, SW35 SW_Push, SW36 SW_Push, SW37 SW_Push, SW38 SW_Push, SW39 SW_Push, SW4 SW_Push, SW40 SW_Push, SW41 SW_Push, SW42 SW_Push, SW43 SW_Push, SW44 SW_Push, SW45 SW_Push, SW46 SW_Push, SW47 SW_Push, SW48 SW_Push, SW49 SW_Push, SW5 SW_Push, SW50 SW_Push, SW51 SW_Push, SW52 SW_Push, SW53 SW_Push, SW54 SW_Push, SW55 SW_Push, SW56 SW_Push, SW57 SW_Push, SW58 SW_Push, SW59 SW_Push, SW6 SW_Push, SW60 SW_Push, SW61 SW_Push, SW7 SW_Push, SW8 SW_Push, SW9 SW_Push

Commit message: values
Parts:
- D1, D2, D3: value D -> THT LED
- D100, D101, D102, D103, D104, D105, D106, D107, D108, D109, D110, D111, D112, D113, D114, D115, D116, D117, D118, D119, D120, D121, D122, D123, D124, D125, D65, D66, D67, D68, D69, D70, D71, D72, D73, D74, D75, D76, D77, D78, D79, D80, D81, D82, D83, D84, D85, D86, D87, D88, D89, D90, D91, D92, D93, D94, D95, D96, D97, D98, D99: value LED -> SMD LED
- SW1, SW10, SW11, SW12, SW13, SW14, SW15, SW16, SW17, SW18, SW19, SW2, SW20, SW21, SW22, SW23, SW24, SW25, SW26, SW27, SW28, SW29, SW3, SW30, SW31, SW32, SW33, SW34, SW35, SW36, SW37, SW38, SW39, SW4, SW40, SW41, SW42, SW43, SW44, SW45, SW46, SW47, SW48, SW49, SW5, SW50, SW51, SW52, SW53, SW54, SW55, SW56, SW57, SW58, SW59, SW6, SW60, SW61, SW7, SW8, SW9: value SW_Push -> Switch

Commit message: mcu connect
Connections:
- net CAPS is gone; now on net SIG2: D2.1 (K)
- net INPUT is gone; now on net SIG3: D3.1 (K)
- net NUM is gone; now on net SIG1: D1.1 (K)
- net BL PWM: now also A1.27 (GPIO21)
- net COL0: now also A1.15 (GPIO11)
- net COL1: now also A1.14 (GPIO10)
- net COL10: now also A1.6 (GPIO4)
- net COL11: now also A1.7 (GPIO5)
- net COL2: now also A1.12 (GPIO9)
- net COL3: now also A1.11 (GPIO8)
- net COL4: now also A1.10 (GPIO7)
- net COL5: now also A1.9 (GPIO6)
- net COL6: now also A1.1 (GPIO0)
- net COL7: now also A1.2 (GPIO1)
- net COL8: now also A1.4 (GPIO2)
- net COL9: now also A1.5 (GPIO3)
- net GND: now also A1.13 (GND), A1.18 (GND), A1.23 (GND), A1.28 (GND), A1.3 (GND), A1.38 (GND), A1.8 (GND)
- net ROW0: now also A1.16 (GPIO12)
- net ROW1: now also A1.17 (GPIO13)
- net ROW2: now also A1.19 (GPIO14)
- net ROW3: now also A1.20 (GPIO15)
- net ROW4: now also A1.21 (GPIO16)
- net ROW5: now also A1.22 (GPIO17)
- net SIG1: now reaches A1.24 (GPIO18)
- net SIG2: now reaches A1.25 (GPIO19)
- net SIG3: now reaches A1.26 (GPIO20)

Commit message: footprints
Parts:
- D1, D2, D3: footprint (none) -> LED_THT:LED_D3.0mm
- D10, D11, D12, D13, D14, D15, D16, D17, D18, D19, D20, D21, D22, D23, D24, D25, D26, D27, D28, D29, D30, D31, D32, D33, D34, D35, D36, D37, D38, D39, D4, D40, D41, D42, D43, D44, D45, D46, D47, D48, D49, D5, D50, D51, D52, D53, D54, D55, D56, D57, D58, D59, D6, D60, D61, D62, D63, D64, D7, D8, D9: footprint (none) -> Diode_SMD:D_SOD-123
- D100, D101, D102, D103, D104, D105, D106, D107, D108, D109, D110, D111, D112, D113, D114, D115, D116, D117, D118, D119, D120, D121, D122, D123, D124, D125, D65, D66, D67, D68, D69, D70, D71, D72, D73, D74, D75, D76, D77, D78, D79, D80, D81, D82, D83, D84, D85, D86, D87, D88, D89, D90, D91, D92, D93, D94, D95, D96, D97, D98, D99: footprint (none) -> LED_SMD:LED_1206_3216Metric_ReverseMount_Hole1.8x2.4mm
- Q1: footprint (none) -> Package_TO_SOT_SMD:SOT-23
- R1, R10, R11, R12, R13, R14, R15, R16, R17, R18, R19, R2, R20, R21, R22, R23, R24, R25, R26, R27, R28, R29, R3, R30, R31, R32, R33, R34, R35, R36, R37, R38, R39, R4, R40, R41, R42, R43, R44, R45, R46, R47, R48, R49, R5, R50, R51, R52, R53, R54, R55, R56, R57, R58, R59, R6, R60, R61, R62, R63, R64, R65, R66, R7, R8, R9: footprint (none) -> Resistor_SMD:R_0603_1608Metric
- SW16: footprint (none) -> Krtkus_lib:KS-33 3.0

Commit message: res
Parts:
- R1, R2, R3: value 160 -> VARTHT; footprint Resistor_SMD:R_0603_1608Metric -> Resistor_THT:R_Axial_DIN0207_L6.3mm_D2.5mm_P10.16mm_Horizontal
Changed lines of the file:
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@@
 			)
 		)
-		(property "Value" "160"
+		(property "Value" "VARTHT"
 			(at 68.58 200.66 90)
 			(do_not_autoplace yes)
@@
 			)
 		)
-		(property "Footprint" "Resistor_SMD:R_0603_1608Metric"
+		(property "Footprint" "Resistor_THT:R_Axial_DIN0207_L6.3mm_D2.5mm_P10.16mm_Horizontal"
 			(at 68.58 198.882 90)
 			(effects
@@
 			)
 		)
-		(property "Value" "160"
+		(property "Value" "VARTHT"
 			(at 68.58 209.55 90)
 			(do_not_autoplace yes)
@@
 			)
 		)
-		(property "Footprint" "Resistor_SMD:R_0603_1608Metric"
+		(property "Footprint" "Resistor_THT:R_Axial_DIN0207_L6.3mm_D2.5mm_P10.16mm_Horizontal"
 			(at 68.58 207.772 90)
 			(effects
@@
 			)
 		)
-		(property "Value" "160"
+		(property "Value" "VARTHT"
 			(at 68.58 191.77 90)
 			(do_not_autoplace yes)
@@
 			)
 		)
-		(property "Footprint" "Resistor_SMD:R_0603_1608Metric"
+		(property "Footprint" "Resistor_THT:R_Axial_DIN0207_L6.3mm_D2.5mm_P10.16mm_Horizontal"
 			(at 68.58 189.992 90)
 			(effects

Commit message: more footprints
Parts:
- D10, D11, D12, D13, D14, D15, D16, D17, D18, D19, D20, D21, D22, D23, D24, D25, D26, D27, D28, D29, D30, D31, D32, D33, D34, D35, D36, D37, D38, D39, D4, D40, D41, D42, D43, D44, D45, D46, D47, D48, D49, D5, D50, D51, D52, D53, D54, D55, D56, D57, D58, D59, D6, D60, D61, D62, D63, D64, D7, D8, D9: value Diode -> D
- R1, R2, R3: value VARTHT -> THT R
- SW1, SW10, SW11, SW12, SW13, SW14, SW15, SW17, SW18, SW19, SW2, SW20, SW21, SW22, SW23, SW24, SW25, SW26, SW27, SW28, SW29, SW3, SW30, SW31, SW32, SW33, SW34, SW35, SW36, SW37, SW38, SW39, SW4, SW40, SW41, SW42, SW43, SW44, SW45, SW46, SW47, SW48, SW49, SW5, SW50, SW51, SW52, SW53, SW54, SW55, SW56, SW57, SW58, SW59, SW6, SW60, SW61, SW7, SW8, SW9: footprint (none) -> Krtkus_lib:KS-33 3.0
