File: source/kicad/Krteq/Krteq.kicad_sch (KiCad schematic)
At the start: 254 parts, among them Q1 Q_NMOS, SW1 Switch, SW10 Switch, SW11 Switch, SW12 Switch, SW13 Switch, SW14 Switch, SW15 Switch, SW16 Switch, SW17 Switch, SW18 Switch, SW19 Switch, SW2 Switch, SW20 Switch, SW21 Switch, SW22 Switch, SW23 Switch, SW24 Switch, SW25 Switch, SW26 Switch, SW27 Switch, SW28 Switch, SW29 Switch, SW3 Switch, SW30 Switch, SW31 Switch, SW32 Switch, SW33 Switch, SW34 Switch, SW35 Switch, SW36 Switch, SW37 Switch, SW38 Switch, SW39 Switch, SW4 Switch, SW40 Switch, SW41 Switch, SW42 Switch, SW43 Switch, SW44 Switch, SW45 Switch, SW46 Switch, SW47 Switch, SW48 Switch, SW49 Switch, SW5 Switch, SW50 Switch, SW51 Switch, SW52 Switch, SW53 Switch, SW54 Switch, SW55 Switch, SW56 Switch, SW57 Switch, SW58 Switch, SW59 Switch, SW6 Switch, SW60 Switch, SW61 Switch, SW7 Switch, SW8 Switch, SW9 Switch

Commit message: name
Parts:
- SW1, SW10, SW11, SW12, SW13, SW14, SW15, SW16, SW17, SW18, SW19, SW2, SW20, SW21, SW22, SW23, SW24, SW25, SW26, SW27, SW28, SW29, SW3, SW30, SW31, SW32, SW33, SW34, SW35, SW36, SW37, SW38, SW39, SW4, SW40, SW41, SW42, SW43, SW44, SW45, SW46, SW47, SW48, SW49, SW5, SW50, SW51, SW52, SW53, SW54, SW55, SW56, SW57, SW58, SW59, SW6, SW60, SW61, SW7, SW8, SW9: footprint Krtkus_lib:KS-33 3.0 -> Krteq_lib:KS-33 3.0

Commit message: switch footprints
Parts:
- SW1, SW10, SW11, SW12, SW13, SW14, SW15, SW16, SW17, SW18, SW19, SW2, SW20, SW21, SW22, SW23, SW24, SW25, SW26, SW27, SW28, SW29, SW3, SW30, SW32, SW33, SW34, SW35, SW36, SW37, SW38, SW39, SW4, SW40, SW41, SW42, SW43, SW44, SW45, SW46, SW47, SW48, SW49, SW5, SW50, SW51, SW52, SW53, SW54, SW55, SW56, SW57, SW58, SW59, SW6, SW60, SW61, SW7, SW8, SW9: footprint Krteq_lib:KS-33 3.0 -> Krteq:KS-33B Hotswap 1u
- SW31: footprint Krteq_lib:KS-33 3.0 -> Krteq:KS-33B Hotswap 2u
Changed lines of the file:
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@@
 			)
 		)
-		(property "Footprint" "Krteq_lib:KS-33 3.0"
+		(property "Footprint" "Krteq:KS-33B Hotswap 1u"
 			(at 228.6 85.09 0)
 			(effects
@@
 			)
 		)
-		(property "Footprint" "Krteq_lib:KS-33 3.0"
+		(property "Footprint" "Krteq:KS-33B Hotswap 1u"
 			(at 215.9 50.8 0)
 			(effects
@@
 			)
 		)
-		(property "Footprint" "Krteq_lib:KS-33 3.0"
+		(property "Footprint" "Krteq:KS-33B Hotswap 1u"
 			(at 279.4 50.8 0)
 			(effects
@@
 			)
 		)
-		(property "Footprint" "Krteq_lib:KS-33 3.0"
+		(property "Footprint" "Krteq:KS-33B Hotswap 1u"
 			(at 203.2 50.8 0)
 			(effects
@@
 			)
 		)
-		(property "Footprint" "Krteq_lib:KS-33 3.0"
+		(property "Footprint" "Krteq:KS-33B Hotswap 1u"
 			(at 304.8 85.09 0)
 			(effects
@@
 			)
 		)
-		(property "Footprint" "Krteq_lib:KS-33 3.0"
+		(property "Footprint" "Krteq:KS-33B Hotswap 1u"
 			(at 215.9 85.09 0)
 			(effects
@@
 			)
 		)
-		(property "Footprint" "Krteq_lib:KS-33 3.0"
+		(property "Footprint" "Krteq:KS-33B Hotswap 1u"
 			(at 203.2 62.23 0)
 			(effects
@@
 			)
 		)
-		(property "Footprint" "Krteq_lib:KS-33 3.0"
+		(property "Footprint" "Krteq:KS-33B Hotswap 1u"
 			(at 228.6 50.8 0)
 			(effects
@@
 			)
 		)
-		(property "Footprint" "Krteq_lib:KS-33 3.0"
+		(property "Footprint" "Krteq:KS-33B Hotswap 1u"
 			(at 279.4 62.23 0)
 			(effects
@@
 			)
 		)
-		(property "Footprint" "Krteq_lib:KS-33 3.0"
+		(property "Footprint" "Krteq:KS-33B Hotswap 1u"
 			(at 254 73.66 0)
 			(effects
@@
 			)
 		)
-		(property "Footprint" "Krteq_lib:KS-33 3.0"
+		(property "Footprint" "Krteq:KS-33B Hotswap 1u"
 			(at 241.3 62.23 0)
 			(effects
@@
 			)
 		)
-		(property "Footprint" "Krteq_lib:KS-33 3.0"
+		(property "Footprint" "Krteq:KS-33B Hotswap 2u"
 			(at 247.65 96.52 0)
 			(effects
@@
 			)
 		)
-		(property "Footprint" "Krteq_lib:KS-33 3.0"
+		(property "Footprint" "Krteq:KS-33B Hotswap 1u"
 			(at 241.3 85.09 0)
 			(effects
@@
 			)
 		)
-		(property "Footprint" "Krteq_lib:KS-33 3.0"
+		(property "Footprint" "Krteq:KS-33B Hotswap 1u"
 			(at 292.1 62.23 0)
 			(effects
@@
 			)
 		)
-		(property "Footprint" "Krteq_lib:KS-33 3.0"
+		(property "Footprint" "Krteq:KS-33B Hotswap 1u"
 			(at 317.5 50.8 0)
 			(effects
@@
 			)
 		)
-		(property "Footprint" "Krteq_lib:KS-33 3.0"
+		(property "Footprint" "Krteq:KS-33B Hotswap 1u"
 			(at 304.8 50.8 0)
 			(effects
@@
 			)
 		)
-		(property "Footprint" "Krteq_lib:KS-33 3.0"
+		(property "Footprint" "Krteq:KS-33B Hotswap 1u"
 			(at 317.5 39.37 0)
 			(effects
@@
 			)
 		)
-		(property "Footprint" "Krteq_lib:KS-33 3.0"
+		(property "Footprint" "Krteq:KS-33B Hotswap 1u"
 			(at 304.8 96.52 0)
 			(effects
@@
 			)
 		)
-		(property "Footprint" "Krteq_lib:KS-33 3.0"
+		(property "Footprint" "Krteq:KS-33B Hotswap 1u"
 			(at 215.9 62.23 0)
 			(effects
@@
 			)
 		)
-		(property "Footprint" "Krteq_lib:KS-33 3.0"
+		(property "Footprint" "Krteq:KS-33B Hotswap 1u"
 			(at 292.1 50.8 0)
 			(effects
@@
 			)
 		)
-		(property "Footprint" "Krteq_lib:KS-33 3.0"
+		(property "Footprint" "Krteq:KS-33B Hotswap 1u"
 			(at 228.6 62.23 0)
 			(effects
@@
 			)
 		)
-		(property "Footprint" "Krteq_lib:KS-33 3.0"
+		(property "Footprint" "Krteq:KS-33B Hotswap 1u"
 			(at 292.1 73.66 0)
 			(effects
@@
 			)
 		)
-		(property "Footprint" "Krteq_lib:KS-33 3.0"
+		(property "Footprint" "Krteq:KS-33B Hotswap 1u"
 			(at 266.7 73.66 0)
 			(effects
@@
 			)
 		)
-		(property "Footprint" "Krteq_lib:KS-33 3.0"
+		(property "Footprint" "Krteq:KS-33B Hotswap 1u"
 			(at 215.9 73.66 0)
 			(effects
@@
 			)
 		)
-		(property "Footprint" "Krteq_lib:KS-33 3.0"
+		(property "Footprint" "Krteq:KS-33B Hotswap 1u"
 			(at 190.5 73.66 0)
 			(effects
@@
 			)
 		)
-		(property "Footprint" "Krteq_lib:KS-33 3.0"
+		(property "Footprint" "Krteq:KS-33B Hotswap 1u"
 			(at 279.4 85.09 0)
 			(effects
@@
 			)
 		)
-		(property "Footprint" "Krteq_lib:KS-33 3.0"
+		(property "Footprint" "Krteq:KS-33B Hotswap 1u"
 			(at 190.5 96.52 0)
 			(effects
@@
 			)
 		)
-		(property "Footprint" "Krteq_lib:KS-33 3.0"
+		(property "Footprint" "Krteq:KS-33B Hotswap 1u"
 			(at 279.4 96.52 0)
 			(effects
@@
 			)
 		)
-		(property "Footprint" "Krteq_lib:KS-33 3.0"
+		(property "Footprint" "Krteq:KS-33B Hotswap 1u"
 			(at 266.7 50.8 0)
 			(effects
@@
 			)
 		)
-		(property "Footprint" "Krteq_lib:KS-33 3.0"
+		(property "Footprint" "Krteq:KS-33B Hotswap 1u"
 			(at 241.3 50.8 0)
 			(effects
@@
 			)
 		)
-		(property "Footprint" "Krteq_lib:KS-33 3.0"
+		(property "Footprint" "Krteq:KS-33B Hotswap 1u"
 			(at 215.9 96.52 0)
 			(effects
@@
 			)
 		)
-		(property "Footprint" "Krteq_lib:KS-33 3.0"
+		(property "Footprint" "Krteq:KS-33B Hotswap 1u"
 			(at 254 62.23 0)
 			(effects
@@
 			)
 		)
-		(property "Footprint" "Krteq_lib:KS-33 3.0"
+		(property "Footprint" "Krteq:KS-33B Hotswap 1u"
 			(at 266.7 96.52 0)
 			(effects
@@
 			)
 		)
-		(property "Footprint" "Krteq_lib:KS-33 3.0"
+		(property "Footprint" "Krteq:KS-33B Hotswap 1u"
 			(at 177.8 85.09 0)
 			(effects
@@
 			)
 		)
-		(property "Footprint" "Krteq_lib:KS-33 3.0"
+		(property "Footprint" "Krteq:KS-33B Hotswap 1u"
 			(at 266.7 85.09 0)
 			(effects
@@
 			)
 		)
-		(property "Footprint" "Krteq_lib:KS-33 3.0"
+		(property "Footprint" "Krteq:KS-33B Hotswap 1u"
 			(at 292.1 96.52 0)
 			(effects
@@
 			)
 		)
-		(property "Footprint" "Krteq_lib:KS-33 3.0"
+		(property "Footprint" "Krteq:KS-33B Hotswap 1u"
 			(at 228.571 96.52 0)
 			(effects
@@
 			)
 		)
-		(property "Footprint" "Krteq_lib:KS-33 3.0"
+		(property "Footprint" "Krteq:KS-33B Hotswap 1u"
 			(at 266.7 62.23 0)
 			(effects
@@
 			)
 		)
-		(property "Footprint" "Krteq_lib:KS-33 3.0"
+		(property "Footprint" "Krteq:KS-33B Hotswap 1u"
 			(at 203.2 85.09 0)
 			(effects
@@
 			)
 		)
-		(property "Footprint" "Krteq_lib:KS-33 3.0"
+		(property "Footprint" "Krteq:KS-33B Hotswap 1u"
 			(at 254 85.09 0)
 			(effects
@@
 			)
 		)
-		(property "Footprint" "Krteq_lib:KS-33 3.0"
+		(property "Footprint" "Krteq:KS-33B Hotswap 1u"
 			(at 177.8 73.66 0)
 			(effects
@@
 			)
 		)
-		(property "Footprint" "Krteq_lib:KS-33 3.0"
+		(property "Footprint" "Krteq:KS-33B Hotswap 1u"
 			(at 177.8 39.37 0)
 			(effects
@@
 			)
 		)
-		(property "Footprint" "Krteq_lib:KS-33 3.0"
+		(property "Footprint" "Krteq:KS-33B Hotswap 1u"
 			(at 177.8 50.8 0)
 			(effects
@@
 			)
 		)
-		(property "Footprint" "Krteq_lib:KS-33 3.0"
+		(property "Footprint" "Krteq:KS-33B Hotswap 1u"
 			(at 292.1 85.09 0)
 			(effects
@@
 			)
 		)
-		(property "Footprint" "Krteq_lib:KS-33 3.0"
+		(property "Footprint" "Krteq:KS-33B Hotswap 1u"
 			(at 228.6 73.66 0)
 			(effects
@@
 			)
 		)
-		(property "Footprint" "Krteq_lib:KS-33 3.0"
+		(property "Footprint" "Krteq:KS-33B Hotswap 1u"
 			(at 241.3 73.66 0)
 			(effects
@@
 			)
 		)
-		(property "Footprint" "Krteq_lib:KS-33 3.0"
+		(property "Footprint" "Krteq:KS-33B Hotswap 1u"
 			(at 254 50.8 0)
 			(effects
@@
 			)
 		)
-		(property "Footprint" "Krteq_lib:KS-33 3.0"
+		(property "Footprint" "Krteq:KS-33B Hotswap 1u"
 			(at 190.5 62.23 0)
 			(effects
@@
 			)
 		)
-		(property "Footprint" "Krteq_lib:KS-33 3.0"
+		(property "Footprint" "Krteq:KS-33B Hotswap 1u"
 			(at 304.8 62.23 0)
 			(effects
@@
 			)
 		)
-		(property "Footprint" "Krteq_lib:KS-33 3.0"
+		(property "Footprint" "Krteq:KS-33B Hotswap 1u"
 			(at 317.5 62.23 0)
 			(effects
@@
 			)
 		)
-		(property "Footprint" "Krteq_lib:KS-33 3.0"
+		(property "Footprint" "Krteq:KS-33B Hotswap 1u"
 			(at 203.171 96.52 0)
 			(effects
@@
 			)
 		)
-		(property "Footprint" "Krteq_lib:KS-33 3.0"
+		(property "Footprint" "Krteq:KS-33B Hotswap 1u"
 			(at 317.5 96.52 0)
 			(effects
@@
 			)
 		)
-		(property "Footprint" "Krteq_lib:KS-33 3.0"
+		(property "Footprint" "Krteq:KS-33B Hotswap 1u"
 			(at 190.5 50.8 0)
 			(effects
@@
 			)
 		)
-		(property "Footprint" "Krteq_lib:KS-33 3.0"
+		(property "Footprint" "Krteq:KS-33B Hotswap 1u"
 			(at 317.5 73.66 0)
 			(effects
@@
 			)
 		)
-		(property "Footprint" "Krteq_lib:KS-33 3.0"
+		(property "Footprint" "Krteq:KS-33B Hotswap 1u"
 			(at 203.2 73.66 0)
 			(effects
@@
 			)
 		)
-		(property "Footprint" "Krteq_lib:KS-33 3.0"
+		(property "Footprint" "Krteq:KS-33B Hotswap 1u"
 			(at 190.5 85.09 0)
 			(effects
@@
 			)
 		)
-		(property "Footprint" "Krteq_lib:KS-33 3.0"
+		(property "Footprint" "Krteq:KS-33B Hotswap 1u"
 			(at 177.8 62.23 0)
 			(effects
@@
 			)
 		)
-		(property "Footprint" "Krteq_lib:KS-33 3.0"
+		(property "Footprint" "Krteq:KS-33B Hotswap 1u"
 			(at 177.8 96.52 0)
 			(effects
@@
 			)
 		)
-		(property "Footprint" "Krteq_lib:KS-33 3.0"
+		(property "Footprint" "Krteq:KS-33B Hotswap 1u"
 			(at 317.5 85.09 0)
 			(effects
@@
 			)
 		)
-		(property "Footprint" "Krteq_lib:KS-33 3.0"
+		(property "Footprint" "Krteq:KS-33B Hotswap 1u"
 			(at 304.8 73.66 0)
 			(effects
@@
 			)
 		)
-		(property "Footprint" "Krteq_lib:KS-33 3.0"
+		(property "Footprint" "Krteq:KS-33B Hotswap 1u"
 			(at 279.4 73.66 0)
 			(effects

Commit message: updates
Parts:
- A1: footprint Module:RaspberryPi_Pico_Common_Unspecified -> Module:RaspberryPi_Pico_Common_THT
Changed lines of the file:
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@@
 			)
 		)
-		(property "Footprint" "Module:RaspberryPi_Pico_Common_Unspecified"
+		(property "Footprint" "Module:RaspberryPi_Pico_Common_THT"
 			(at 76.2 133.35 0)
 			(effects

Commit message: update
Parts:
- R1, R2, R3: value THT R -> R
Changed lines of the file:
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@@
 			)
 		)
-		(property "Value" "THT R"
+		(property "Value" "R"
 			(at 68.58 200.66 90)
 			(do_not_autoplace yes)
@@
 			)
 		)
-		(property "Value" "THT R"
+		(property "Value" "R"
 			(at 68.58 209.55 90)
 			(do_not_autoplace yes)
@@
 			)
 		)
-		(property "Value" "THT R"
+		(property "Value" "R"
 			(at 68.58 191.77 90)
 			(do_not_autoplace yes)

Commit message: update
Parts:
- removed Q1: Q_NMOS, Package_TO_SOT_SMD:SOT-23, symbol Device:Q_NMOS
- added Q1: Q_NMOS_GSD, Package_TO_SOT_SMD:SOT-23, symbol Transistor_FET:Q_NMOS_GSD
- D100, D101, D102, D103, D104, D105, D106, D107, D108, D109, D110, D111, D112, D113, D114, D115, D116, D117, D118, D119, D120, D121, D122, D123, D124, D125, D65, D66, D67, D68, D69, D70, D71, D72, D73, D74, D75, D76, D77, D78, D79, D80, D81, D82, D83, D84, D85, D86, D87, D88, D89, D90, D91, D92, D93, D94, D95, D96, D97, D98, D99: footprint LED_SMD:LED_1206_3216Metric_ReverseMount_Hole1.8x2.4mm -> Krteq:MHT151WDT
- R10, R11, R12, R13, R14, R15, R16, R17, R18, R19, R20, R21, R22, R23, R24, R25, R26, R27, R28, R29, R30, R31, R32, R33, R34, R35, R36, R37, R38, R39, R4, R40, R41, R42, R43, R44, R45, R46, R47, R48, R49, R5, R50, R51, R52, R53, R54, R55, R56, R57, R58, R59, R6, R60, R61, R62, R63, R64, R7, R8, R9: value 470 -> 330
Connections:
- net BL DRAIN: now also Q1.3 (D)
- net GND: now also Q1.2 (S)
- net at R65.1, R66.1: now also Q1.1 (G)

Commit message: pcb update
Parts:
- renumbered SW13 to SW12, SW14 to SW13, SW15 to SW14, SW16 to SW15, SW12 to SW16, SW23 to SW22, SW24 to SW23, SW25 to SW24, SW26 to SW25, SW22 to SW26
Connections:
- net COL2: now also SW16.2
- net at D19.2 (A): now also SW16.1
Changed lines of the file:
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@@
 	(wire
 		(pts
-			(xy 233.651 100.33) (xy 233.651 101.6)
-		)
-		(stroke
-			(width 0)
-			(type default)
-		)
-	)
-	(wire
-		(pts
 			(xy 259.08 78.74) (xy 259.08 90.17)
 		)
@@
 	(wire
 		(pts
-			(xy 223.491 101.6) (xy 223.52 101.6)
-		)
-		(stroke
-			(width 0)
-			(type default)
-		)
-	)
-	(wire
-		(pts
 			(xy 236.22 86.36) (xy 248.92 86.36)
 		)
@@
 	(wire
 		(pts
+			(xy 233.68 90.17) (xy 233.68 101.6)
+		)
+		(stroke
+			(width 0)
+			(type default)
+		)
+	)
+	(wire
+		(pts
 			(xy 210.82 86.36) (xy 223.52 86.36)
 		)
@@
 	(wire
 		(pts
-			(xy 233.68 100.33) (xy 233.68 90.17)
-		)
-		(stroke
-			(width 0)
-			(type default)
-		)
-	)
-	(wire
-		(pts
 			(xy 222.25 205.74) (xy 228.6 205.74)
 		)
@@
 	(wire
 		(pts
-			(xy 233.651 100.33) (xy 233.68 100.33)
-		)
-		(stroke
-			(width 0)
-			(type default)
-		)
-	)
-	(wire
-		(pts
 			(xy 62.23 200.66) (xy 62.23 191.77)
 		)
@@
 		(dnp no)
 		(fields_autoplaced yes)
-		(property "Reference" "SW26"
+		(property "Reference" "SW25"
 			(at 228.6 92.202 0)
 			(do_not_autoplace yes)
@@
 			(project "Krteq"
 				(path "/9e7f33ad-d3b4-42c3-9373-23856f560db6"
-					(reference "SW26")
+					(reference "SW25")
 					(unit 1)
 				)
@@
 		(dnp no)
 		(fields_autoplaced yes)
-		(property "Reference" "SW13"
+		(property "Reference" "SW12"
 			(at 203.2 57.912 0)
 			(do_not_autoplace yes)
@@
 			(project "Krteq"
 				(path "/9e7f33ad-d3b4-42c3-9373-23856f560db6"
-					(reference "SW13")
+					(reference "SW12")
 					(unit 1)
 				)
@@
 		(dnp no)
 		(fields_autoplaced yes)
-		(property "Reference" "SW14"
+		(property "Reference" "SW13"
 			(at 203.2 69.342 0)
 			(do_not_autoplace yes)
@@
 			(project "Krteq"
 				(path "/9e7f33ad-d3b4-42c3-9373-23856f560db6"
-					(reference "SW14")
+					(reference "SW13")
 					(unit 1)
 				)
@@
 		(dnp no)
 		(fields_autoplaced yes)
-		(property "Reference" "SW23"
+		(property "Reference" "SW22"
 			(at 228.6 57.912 0)
 			(do_not_autoplace yes)
@@
 			(project "Krteq"
 				(path "/9e7f33ad-d3b4-42c3-9373-23856f560db6"
-					(reference "SW23")
+					(reference "SW22")
 					(unit 1)
 				)
@@
 		(dnp no)
 		(fields_autoplaced yes)
-		(property "Reference" "SW24"
+		(property "Reference" "SW23"
 			(at 228.6 69.342 0)
 			(do_not_autoplace yes)
@@
 			(project "Krteq"
 				(path "/9e7f33ad-d3b4-42c3-9373-23856f560db6"
-					(reference "SW24")
+					(reference "SW23")
 					(unit 1)
 				)
@@
 	(symbol
 		(lib_id "Switch:SW_Push")
-		(at 228.571 101.6 0)
+		(at 228.6 101.6 0)
 		(unit 1)
 		(exclude_from_sim no)
@@
 		(dnp no)
 		(fields_autoplaced yes)
-		(property "Reference" "SW22"
-			(at 228.571 103.632 0)
+		(property "Reference" "SW26"
+			(at 228.6 103.632 0)
 			(do_not_autoplace yes)
 			(effects
@@
 		)
 		(property "Value" "Switch"
-			(at 228.571 103.124 0)
+			(at 228.6 103.124 0)
 			(do_not_autoplace yes)
 			(effects
@@
 		)
 		(property "Footprint" "Krteq:KS-33B Hotswap 1u"
-			(at 228.571 96.52 0)
+			(at 228.6 96.52 0)
 			(effects
 				(font
@@
 		)
 		(property "Datasheet" "~"
-			(at 228.571 96.52 0)
+			(at 228.6 96.52 0)
 			(effects
 				(font
@@
 		)
 		(property "Description" "Push button switch, generic, two pins"
-			(at 228.571 101.6 0)
+			(at 228.6 101.6 0)
 			(effects
 				(font
@@
 			(project "Krteq"
 				(path "/9e7f33ad-d3b4-42c3-9373-23856f560db6"
-					(reference "SW22")
+					(reference "SW26")
 					(unit 1)
 				)
@@
 		(dnp no)
 		(fields_autoplaced yes)
-		(property "Reference" "SW16"
+		(property "Reference" "SW15"
 			(at 203.2 92.202 0)
 			(do_not_autoplace yes)
@@
 			(project "Krteq"
 				(path "/9e7f33ad-d3b4-42c3-9373-23856f560db6"
-					(reference "SW16")
+					(reference "SW15")
 					(unit 1)
 				)
@@
 		(dnp no)
 		(fields_autoplaced yes)
-		(property "Reference" "SW25"
+		(property "Reference" "SW24"
 			(at 228.6 80.772 0)
 			(do_not_autoplace yes)
@@
 			(project "Krteq"
 				(path "/9e7f33ad-d3b4-42c3-9373-23856f560db6"
-					(reference "SW25")
+					(reference "SW24")
 					(unit 1)
 				)
@@
 	(symbol
 		(lib_id "Switch:SW_Push")
-		(at 203.171 101.6 0)
+		(at 203.2 101.6 0)
 		(unit 1)
 		(exclude_from_sim no)
@@
 		(dnp no)
 		(fields_autoplaced yes)
-		(property "Reference" "SW12"
-			(at 203.171 103.632 0)
+		(property "Reference" "SW16"
+			(at 203.2 103.632 0)
 			(do_not_autoplace yes)
 			(effects
@@
 		)
 		(property "Value" "Switch"
-			(at 203.171 103.124 0)
+			(at 203.2 103.124 0)
 			(do_not_autoplace yes)
 			(effects
@@
 		)
 		(property "Footprint" "Krteq:KS-33B Hotswap 1u"
-			(at 203.171 96.52 0)
+			(at 203.2 96.52 0)
 			(effects
 				(font
@@
 		)
 		(property "Datasheet" "~"
-			(at 203.171 96.52 0)
+			(at 203.2 96.52 0)
 			(effects
 				(font
@@
 		)
 		(property "Description" "Push button switch, generic, two pins"
-			(at 203.171 101.6 0)
+			(at 203.2 101.6 0)
 			(effects
 				(font
@@
 			(project "Krteq"
 				(path "/9e7f33ad-d3b4-42c3-9373-23856f560db6"
-					(reference "SW12")
+					(reference "SW16")
 					(unit 1)
 				)
@@
 		(dnp no)
 		(fields_autoplaced yes)
-		(property "Reference" "SW15"
+		(property "Reference" "SW14"
 			(at 203.2 80.772 0)
 			(do_not_autoplace yes)
@@
 			(project "Krteq"
 				(path "/9e7f33ad-d3b4-42c3-9373-23856f560db6"
-					(reference "SW15")
+					(reference "SW14")
 					(unit 1)
 				)
