File: source/kicad/Krteq/Krteq.kicad_sch (KiCad schematic)
At the start: 263 parts, among them Q1 Q NMOS GSD, Q2 Q NMOS GSD, Q3 Q NMOS GSD, Q4 Q NMOS GSD, SW1 Switch, SW10 Switch, SW11 Switch, SW12 Switch, SW13 Switch, SW14 Switch, SW15 Switch, SW16 Switch, SW17 Switch, SW18 Switch, SW19 Switch, SW2 Switch, SW20 Switch, SW21 Switch, SW22 Switch, SW23 Switch, SW24 Switch, SW25 Switch, SW26 Switch, SW27 Switch, SW28 Switch, SW29 Switch, SW3 Switch, SW30 Switch, SW31 Switch, SW32 Switch, SW33 Switch, SW34 Switch, SW35 Switch, SW36 Switch, SW37 Switch, SW38 Switch, SW39 Switch, SW4 Switch, SW40 Switch, SW41 Switch, SW42 Switch, SW43 Switch, SW44 Switch, SW45 Switch, SW46 Switch, SW47 Switch, SW48 Switch, SW49 Switch, SW5 Switch, SW50 Switch, SW51 Switch, SW52 Switch, SW53 Switch, SW54 Switch, SW55 Switch, SW56 Switch, SW57 Switch, SW58 Switch, SW59 Switch, SW6 Switch, SW60 Switch, SW61 Switch, SW7 Switch, SW8 Switch, SW9 Switch

Commit message: update
Parts:
- removed D1, D100, D101, D102, D103, D104, D105, D106, D107, D108, D109, D110, D111, D112, D113, D114, D115, D116, D117, D118, D119, D120, D121, D122, D123, D124, D125, D2, D3, D65, D66, D67, D68, D69, D70, D71, D72, D73, D74, D75, D76, D77, D78, D79, D80, D81, D82, D83, D84, D85, D86, D87, D88, D89, D90, D91, D92, D93, D94, D95, D96, D97, D98, D99: LED, Krteq:MHT151WDT, symbol Device:LED
- removed Q1, Q2, Q3, Q4: Q NMOS GSD, Package_TO_SOT_SMD:SOT-23, symbol Transistor_FET:Q_NMOS_GSD
- removed R1, R4, R7: 82Ω, Resistor_SMD:R_0603_1608Metric, symbol Device:R
- removed R100, R101, R102, R103, R104, R105, R106, R107, R108, R109, R110, R111, R112, R113, R114, R115, R116, R117, R118, R119, R120, R121, R122, R123, R124, R125, R65, R66, R67, R68, R69, R70, R71, R72, R73, R74, R75, R76, R77, R78, R79, R80, R81, R82, R83, R84, R85, R86, R87, R88, R89, R90, R91, R92, R93, R94, R95, R96, R97, R98, R99: 330Ω, Resistor_SMD:R_0603_1608Metric, symbol Device:R
- removed R2, R5: 470Ω, Resistor_SMD:R_0603_1608Metric, symbol Device:R
- removed R3, R6: 10kΩ, Resistor_SMD:R_0603_1608Metric, symbol Device:R
- added C4: 0.47µF, symbol Device:C_Small
- added J71: OLED 128x32, Connector_PinHeader_2.54mm:PinHeader_1x04_P2.54mm_Vertical, symbol Connector:Conn_01x04_Pin
- added R12: 2kΩ, Resistor_SMD:R_0603_1608Metric, symbol Device:R
- added U71: IS31FL3733-QF, Package_DFN_QFN:QFN-48-1EP_6x6mm_P0.4mm_EP4.2x4.2mm, symbol Driver_LED:IS31FL3733-QF
- R10: value 470Ω -> 100kΩ
- R11, R9: value 10kΩ -> 100kΩ; MPN 0603WAF1002T5E -> 0603WAF4700T5E
- R8: value 470Ω -> 20kΩ
Connections:
- net COL0: no longer A1.5 (GPIO3)
- net COL1: no longer A1.6 (GPIO4)
- net COL10: no longer A1.21 (GPIO16)
- net COL11: no longer A1.22 (GPIO17)
- net COL2: no longer A1.7 (GPIO5)
- net COL3: no longer A1.9 (GPIO6)
- net COL4: no longer A1.10 (GPIO7)
- net COL5: no longer A1.29 (GPIO22)
- net COL6: no longer A1.31 (GPIO26_ADC0)
- net COL7: no longer A1.32 (GPIO27_ADC1)
- net COL8: no longer A1.34 (GPIO28_ADC2)
- net COL9: no longer A1.27 (GPIO21)
- net GND: now also C4.2, J71.1 (Pin_1), U71.12 (PGND), U71.34 (AGND), U71.48 (GND), U71.49 (GND), U71.5 (PGND); no longer R11.2
- net ROW0: no longer A1.24 (GPIO18)
- net ROW1: no longer A1.25 (GPIO19)
- net ROW2: no longer A1.16 (GPIO12)
- net ROW3: no longer A1.15 (GPIO11)
- net ROW4: no longer A1.14 (GPIO10)
- net ROW5: no longer A1.12 (GPIO9)
- net VBUS: now also J71.2 (Pin_2)
- net at R8.1: now also U71.35 (RSET); no longer R9.1
- net RGB SDA: now reaches A1.19 (GPIO14)
- net RGB SDA: now also R12.2, U71.41 (SDA)
- net RGB SCL: now reaches A1.20 (GPIO15)
- net RGB SCL: now also R11.2, U71.42 (SCL)
- net 3V3: now reaches A1.36 (3V3)
- net 3V3: now also R11.1, C4.1, R12.1, U71.39 (VIO)
- net RGB SDB: now reaches R10.1
- net RGB SDB: now also A1.15 (GPIO11), U71.46 (~{SDB}); no longer R11.1
- net BL PWM: no longer names the net of R10.2
- net BL PWM: now also R8.2, U71.43 (ADDR1), U71.44 (ADDR2); no longer A1.17 (GPIO13)
- net SIG1: no longer names the net of A1.1 (GPIO0)
- net SIG2: no longer names the net of A1.2 (GPIO1)
- net SIG3: no longer names the net of A1.4 (GPIO2)
- net SIG3: no longer R8.2
- new net: R9.1, U71.47 (IICRST)
- new net CS1: U71.16 (CS1)
- new net CS10: U71.26 (CS10)
- new net CS11: U71.27 (CS11)
- new net CS12: U71.28 (CS12)
- new net CS13: U71.30 (CS13)
- new net CS14: U71.31 (CS14)
- new net CS15: U71.32 (CS15)
- new net CS16: U71.33 (CS16)
- new net CS2: U71.17 (CS2)
- new net CS3: U71.18 (CS3)
- new net CS4: U71.19 (CS4)
- new net CS5: U71.21 (CS5)
- new net CS6: U71.22 (CS6)
- new net CS7: U71.23 (CS7)
- new net CS8: U71.24 (CS8)
- new net CS9: U71.25 (CS9)
- new net OLED SCL: A1.17 (GPIO13), J71.3 (Pin_3)
- new net OLED SDA: A1.16 (GPIO12), J71.4 (Pin_4)
- new net SW1: U71.2 (SW1)
- new net SW10: U71.13 (SW10)
- new net SW11: U71.14 (SW11)
- new net SW2: U71.3 (SW2)
- new net SW3: U71.4 (SW3)
- new net SW4: U71.6 (SW4)
- new net SW5: U71.7 (SW5)
- new net SW6: U71.8 (SW6)
- new net SW7: U71.9 (SW7)
- new net SW8: U71.10 (SW8)
- new net SW9: U71.11 (SW9)
Other:
- note added: "RGB driver"
- note added: "RGB matrix"
- note removed: "Backlight"
- note removed: "Indicators"
- moved on the sheet: A1

Commit message: update
Other:
- note added: "Display interface"
- moved on the sheet: A1, C4, D10, D11, D12, D13, D14, D15, D16, D17, D18, D19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

Commit message: update
Parts:
- added C10, C6, C8: 0.1µF, symbol Device:C_Small
- added C5, C7, C9: 0.47µF, symbol Device:C_Small
Connections:
- net GND: now also C10.2, C5.2, C6.2, C7.2, C8.2, C9.2
- net VBUS: now also U71.20 (PVCC), U71.29 (PVCC), U71.37 (AVCC), U71.38 (DVCC), C10.1, C5.1, C6.1, C7.1, C8.1, C9.1

Commit message: update
Parts:
- added D100, D101, D102, D103, D104, D105, D106, D107, D108, D109, D110, D111, D112, D113, D114, D115, D116, D117, D118, D119, D120, D121, D122, D123, D124, D125, D126, D127, D128, D65, D66, D67, D68, D69, D70, D71, D72, D73, D74, D75, D76, D77, D78, D79, D80, D81, D82, D83, D84, D85, D86, D87, D88, D89, D90, D91, D92, D93, D94, D95, D96, D97, D98, D99: LED_ABGR, symbol Device:LED_ABGR
Connections:
- net CS1: now also D113.1 (A), D65.1 (A), D81.1 (A), D97.1 (A)
- net CS10: now also D106.1 (A), D122.1 (A), D74.1 (A), D90.1 (A)
- net CS11: now also D107.1 (A), D123.1 (A), D75.1 (A), D91.1 (A)
- net CS12: now also D108.1 (A), D124.1 (A), D76.1 (A), D92.1 (A)
- net CS13: now also D109.1 (A), D125.1 (A), D77.1 (A), D93.1 (A)
- net CS14: now also D110.1 (A), D126.1 (A), D78.1 (A), D94.1 (A)
- net CS15: now also D111.1 (A), D127.1 (A), D79.1 (A), D95.1 (A)
- net CS16: now also D112.1 (A), D128.1 (A), D80.1 (A), D96.1 (A)
- net CS2: now also D114.1 (A), D66.1 (A), D82.1 (A), D98.1 (A)
- net CS3: now also D115.1 (A), D67.1 (A), D83.1 (A), D99.1 (A)
- net CS4: now also D100.1 (A), D116.1 (A), D68.1 (A), D84.1 (A)
- net CS5: now also D101.1 (A), D117.1 (A), D69.1 (A), D85.1 (A)
- net CS6: now also D102.1 (A), D118.1 (A), D70.1 (A), D86.1 (A)
- net CS7: now also D103.1 (A), D119.1 (A), D71.1 (A), D87.1 (A)
- net CS8: now also D104.1 (A), D120.1 (A), D72.1 (A), D88.1 (A)
- net CS9: now also D105.1 (A), D121.1 (A), D73.1 (A), D89.1 (A)
- net SW1: now also D65.4 (RK), D66.4 (RK), D67.4 (RK), D68.4 (RK), D69.4 (RK), D70.4 (RK), D71.4 (RK), D72.4 (RK), D73.4 (RK), D74.4 (RK), D75.4 (RK), D76.4 (RK), D77.4 (RK), D78.4 (RK), D79.4 (RK), D80.4 (RK)
- net SW10: now also D113.4 (RK), D114.4 (RK), D115.4 (RK), D116.4 (RK), D117.4 (RK), D118.4 (RK), D119.4 (RK), D120.4 (RK), D121.4 (RK), D122.4 (RK), D123.4 (RK), D124.4 (RK), D125.4 (RK), D126.4 (RK), D127.4 (RK), D128.4 (RK)
- net SW11: now also D113.3 (GK), D114.3 (GK), D115.3 (GK), D116.3 (GK), D117.3 (GK), D118.3 (GK), D119.3 (GK), D120.3 (GK), D121.3 (GK), D122.3 (GK), D123.3 (GK), D124.3 (GK), D125.3 (GK), D126.3 (GK), D127.3 (GK), D128.3 (GK)
- net SW12: now also D113.2 (BK), D114.2 (BK), D115.2 (BK), D116.2 (BK), D117.2 (BK), D118.2 (BK), D119.2 (BK), D120.2 (BK), D121.2 (BK), D122.2 (BK), D123.2 (BK), D124.2 (BK), D125.2 (BK), D126.2 (BK), D127.2 (BK), D128.2 (BK)
- net SW2: now also D65.3 (GK), D66.3 (GK), D67.3 (GK), D68.3 (GK), D69.3 (GK), D70.3 (GK), D71.3 (GK), D72.3 (GK), D73.3 (GK), D74.3 (GK), D75.3 (GK), D76.3 (GK), D77.3 (GK), D78.3 (GK), D79.3 (GK), D80.3 (GK)
- net SW3: now also D65.2 (BK), D66.2 (BK), D67.2 (BK), D68.2 (BK), D69.2 (BK), D70.2 (BK), D71.2 (BK), D72.2 (BK), D73.2 (BK), D74.2 (BK), D75.2 (BK), D76.2 (BK), D77.2 (BK), D78.2 (BK), D79.2 (BK), D80.2 (BK)
- net SW4: now also D81.4 (RK), D82.4 (RK), D83.4 (RK), D84.4 (RK), D85.4 (RK), D86.4 (RK), D87.4 (RK), D88.4 (RK), D89.4 (RK), D90.4 (RK), D91.4 (RK), D92.4 (RK), D93.4 (RK), D94.4 (RK), D95.4 (RK), D96.4 (RK)
- net SW5: now also D81.3 (GK), D82.3 (GK), D83.3 (GK), D84.3 (GK), D85.3 (GK), D86.3 (GK), D87.3 (GK), D88.3 (GK), D89.3 (GK), D90.3 (GK), D91.3 (GK), D92.3 (GK), D93.3 (GK), D94.3 (GK), D95.3 (GK), D96.3 (GK)
- net SW6: now also D81.2 (BK), D82.2 (BK), D83.2 (BK), D84.2 (BK), D85.2 (BK), D86.2 (BK), D87.2 (BK), D88.2 (BK), D89.2 (BK), D90.2 (BK), D91.2 (BK), D92.2 (BK), D93.2 (BK), D94.2 (BK), D95.2 (BK), D96.2 (BK)
- net SW7: now also D100.4 (RK), D101.4 (RK), D102.4 (RK), D103.4 (RK), D104.4 (RK), D105.4 (RK), D106.4 (RK), D107.4 (RK), D108.4 (RK), D109.4 (RK), D110.4 (RK), D111.4 (RK), D112.4 (RK), D97.4 (RK), D98.4 (RK), D99.4 (RK)
- net SW8: now also D100.3 (GK), D101.3 (GK), D102.3 (GK), D103.3 (GK), D104.3 (GK), D105.3 (GK), D106.3 (GK), D107.3 (GK), D108.3 (GK), D109.3 (GK), D110.3 (GK), D111.3 (GK), D112.3 (GK), D97.3 (GK), D98.3 (GK), D99.3 (GK)
- net SW9: now also D100.2 (BK), D101.2 (BK), D102.2 (BK), D103.2 (BK), D104.2 (BK), D105.2 (BK), D106.2 (BK), D107.2 (BK), D108.2 (BK), D109.2 (BK), D110.2 (BK), D111.2 (BK), D112.2 (BK), D97.2 (BK), D98.2 (BK), D99.2 (BK)
Other:
- moved on the sheet: C10, C4, C5, C6, C7, C8, C9, D10, D11, D12, D13, D14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

Commit message: update
Parts:
- removed D112, D128, D96: LED_ABGR, symbol Device:LED_ABGR
- renumbered D121 to D100, D74 to D101, D90 to D102, D106 to D103, D122 to D104, D75 to D105, D91 to D106, D123 to D108, D76 to D109, D92 to D110, D108 to D111, D124 to D112, D77 to D113, D93 to D114, D109 to D115, D125 to D116, D78 to D117, D94 to D118, D110 to D119, D126 to D120, D79 to D121, D95 to D122, D111 to D123, D127 to D124, D80 to D125, D81 to D66, D97 to D67, D113 to D68, D66 to D69, D82 to D70, D98 to D71, D114 to D72, D67 to D73, D83 to D74, D99 to D75, D115 to D76, D68 to D77, D84 to D78, D100 to D79, D116 to D80, D69 to D81, D85 to D82, D101 to D83, D117 to D84, D70 to D85, D102 to D87, D118 to D88, D71 to D89, D87 to D90, D103 to D91, D119 to D92, D72 to D93, D88 to D94, D104 to D95, D120 to D96, D73 to D97, D89 to D98, D105 to D99
Connections:
- net SW12: now also U71.15 (SW12)
Other:
- moved on the sheet: C10, C4, C5, C6, C7, C8, C9, D100, D101, D102, D103, D104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

Commit message: update
Parts:
- R11: value 100kΩ -> 2kΩ
- renumbered D4 to D1, D13 to D10, D14 to D11, D15 to D12, D16 to D13, D17 to D14, D18 to D15, D19 to D16, D20 to D17, D21 to D18, D22 to D19, D5 to D2, D23 to D20, D24 to D21, D25 to D22, D26 to D23, D27 to D24, D28 to D25, D29 to D26, D30 to D27, D31 to D28, D32 to D29, D6 to D3, D33 to D30, D34 to D31, D35 to D32, D36 to D33, D37 to D34, D38 to D35, D39 to D36, D40 to D37, D41 to D38, D42 to D39, D7 to D4, D43 to D40, D44 to D41, D45 to D42, D46 to D43, D47 to D44, D48 to D45, D49 to D46, D50 to D47, D51 to D48, D52 to D49, D8 to D5, D53 to D50, D54 to D51, D55 to D52, D56 to D53, D57 to D54, D58 to D55, D59 to D56, D60 to D57, D61 to D58, D62 to D59, D9 to D6, D63 to D60, D64 to D61, D10 to D7, D11 to D8, D12 to D9
Connections:
- net RGB SCL is gone; now on net SCL: A1.20 (GPIO15), R11.2, U71.42 (SCL)
- net 3V3: now also J71.2 (Pin_2)
- net VBUS: no longer J71.2 (Pin_2)
- net OLED SCL renamed SCL
- net SCL: no longer A1.17 (GPIO13)
- net OLED SDA: no longer names the net of A1.16 (GPIO12)
- net OLED SDA: no longer J71.4 (Pin_4)
- net RGB SDA renamed SDA
- net SDA: now also J71.4 (Pin_4)
- net RGB SDB renamed SDB
- net SDB: now also A1.17 (GPIO13); no longer A1.15 (GPIO11)
Other:
- moved on the sheet: C10, C4, C5, C6, C7, C8, C9, R11, R12, R9

Commit message: update
Parts:
- renumbered C9 to C1, C7 to C2, C5 to C3, C10 to C4, C8 to C5, C4 to C7, R11 to R1, R12 to R2, R10 to R3, R9 to R4, R8 to R5
Changed lines of the file:
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@@
 	(global_label "3V3"
 		(shape input)
-		(at 166.37 265.43 180)
+		(at 166.37 266.7 180)
 		(fields_autoplaced yes)
 		(effects
@@
 		)
 		(property "Intersheetrefs" "${INTERSHEET_REFS}"
-			(at 159.8772 265.43 0)
+			(at 159.8772 266.7 0)
 			(hide yes)
 			(show_name no)
@@
 	(global_label "SCL"
 		(shape input)
-		(at 166.37 262.89 180)
+		(at 166.37 264.16 180)
 		(fields_autoplaced yes)
 		(effects
@@
 		)
 		(property "Intersheetrefs" "${INTERSHEET_REFS}"
-			(at 159.8772 262.89 0)
+			(at 159.8772 264.16 0)
 			(hide yes)
 			(show_name no)
@@
 	(global_label "SDA"
 		(shape input)
-		(at 166.37 260.35 180)
+		(at 166.37 261.62 180)
 		(fields_autoplaced yes)
 		(effects
@@
 		)
 		(property "Intersheetrefs" "${INTERSHEET_REFS}"
-			(at 159.8167 260.35 0)
+			(at 159.8167 261.62 0)
 			(hide yes)
 			(show_name no)
@@
 	(symbol
 		(lib_id "Connector:Conn_01x04_Pin")
-		(at 171.45 265.43 180)
+		(at 171.45 266.7 180)
 		(unit 1)
 		(body_style 1)
@@
 		(dnp no)
 		(property "Reference" "J71"
-			(at 170.815 273.05 0)
-			(hide yes)
+			(at 165.862 254.762 0)
 			(show_name no)
 			(do_not_autoplace no)
@@
 		)
 		(property "Value" "OLED 128x32"
-			(at 165.862 256.286 0)
+			(at 165.862 257.556 0)
 			(show_name no)
 			(do_not_autoplace no)
@@
 		)
 		(property "Footprint" "Connector_PinHeader_2.54mm:PinHeader_1x04_P2.54mm_Vertical"
-			(at 171.45 265.43 0)
+			(at 171.45 266.7 0)
 			(hide yes)
 			(show_name no)
@@
 		)
 		(property "Datasheet" ""
-			(at 171.45 265.43 0)
+			(at 171.45 266.7 0)
 			(hide yes)
 			(show_name no)
@@
 		)
 		(property "Description" "Generic connector, single row, 01x04, script generated"
-			(at 171.45 265.43 0)
+			(at 171.45 266.7 0)
 			(hide yes)
 			(show_name no)
@@
 		(dnp no)
 		(fields_autoplaced yes)
-		(property "Reference" "R8"
+		(property "Reference" "R5"
 			(at 63.5 204.724 90)
 			(show_name no)
@@
 			(project "Krteq"
 				(path "/9e7f33ad-d3b4-42c3-9373-23856f560db6"
-					(reference "R8")
+					(reference "R5")
 					(unit 1)
 				)
@@
 	(symbol
 		(lib_id "power:GND")
-		(at 166.37 267.97 0)
+		(at 166.37 269.24 0)
 		(unit 1)
 		(body_style 1)
@@
 		(fields_autoplaced yes)
 		(property "Reference" "#PWR03"
-			(at 166.37 274.32 0)
+			(at 166.37 275.59 0)
 			(hide yes)
 			(show_name no)
@@
 		)
 		(property "Value" "GND"
-			(at 166.37 273.05 0)
+			(at 166.37 274.32 0)
 			(show_name no)
 			(do_not_autoplace no)
@@
 		)
 		(property "Footprint" ""
-			(at 166.37 267.97 0)
+			(at 166.37 269.24 0)
 			(hide yes)
 			(show_name no)
@@
 		)
 		(property "Datasheet" ""
-			(at 166.37 267.97 0)
+			(at 166.37 269.24 0)
 			(hide yes)
 			(show_name no)
@@
 		)
 		(property "Description" "Power symbol creates a global label with name \"GND\" , ground"
-			(at 166.37 267.97 0)
+			(at 166.37 269.24 0)
 			(hide yes)
 			(show_name no)
@@
 		(in_pos_files yes)
 		(dnp no)
-		(property "Reference" "C5"
+		(property "Reference" "C3"
 			(at 101.6063 152.4 90)
 			(show_name no)
@@
 			(project "Krteq"
 				(path "/9e7f33ad-d3b4-42c3-9373-23856f560db6"
-					(reference "C5")
+					(reference "C3")
 					(unit 1)
 				)
@@
 		(dnp no)
 		(fields_autoplaced yes)
-		(property "Reference" "R12"
+		(property "Reference" "R2"
 			(at 52.324 182.88 90)
 			(show_name no)
@@
 			(project "Krteq"
 				(path "/9e7f33ad-d3b4-42c3-9373-23856f560db6"
-					(reference "R12")
+					(reference "R2")
 					(unit 1)
 				)
@@
 		(dnp no)
 		(fields_autoplaced yes)
-		(property "Reference" "R10"
+		(property "Reference" "R3"
 			(at 45.974 203.2 90)
 			(show_name no)
@@
 			(project "Krteq"
 				(path "/9e7f33ad-d3b4-42c3-9373-23856f560db6"
-					(reference "R10")
+					(reference "R3")
 					(unit 1)
 				)
@@
 		(in_pos_files yes)
 		(dnp no)
-		(property "Reference" "C8"
+		(property "Reference" "C5"
 			(at 91.4463 161.29 90)
 			(show_name no)
@@
 			(project "Krteq"
 				(path "/9e7f33ad-d3b4-42c3-9373-23856f560db6"
-					(reference "C8")
+					(reference "C5")
 					(unit 1)
 				)
@@
 		(in_pos_files yes)
 		(dnp no)
-		(property "Reference" "C4"
+		(property "Reference" "C7"
 			(at 63.5063 171.45 90)
 			(show_name no)
@@
 			(project "Krteq"
 				(path "/9e7f33ad-d3b4-42c3-9373-23856f560db6"
-					(reference "C4")
+					(reference "C7")
 					(unit 1)
 				)
@@
 		(dnp no)
 		(fields_autoplaced yes)
-		(property "Reference" "R11"
+		(property "Reference" "R1"
 			(at 45.974 182.88 90)
 			(show_name no)
@@
 			(project "Krteq"
 				(path "/9e7f33ad-d3b4-42c3-9373-23856f560db6"
-					(reference "R11")
+					(reference "R1")
 					(unit 1)
 				)
@@
 		(in_pos_files yes)
 		(dnp no)
-		(property "Reference" "C9"
+		(property "Reference" "C1"
 			(at 81.2863 152.4 90)
 			(show_name no)
@@
 			(project "Krteq"
 				(path "/9e7f33ad-d3b4-42c3-9373-23856f560db6"
-					(reference "C9")
+					(reference "C1")
 					(unit 1)
 				)
@@
 		(dnp no)
 		(fields_autoplaced yes)
-		(property "Reference" "R9"
+		(property "Reference" "R4"
 			(at 52.324 204.47 90)
 			(show_name no)
@@
 			(project "Krteq"
 				(path "/9e7f33ad-d3b4-42c3-9373-23856f560db6"
-					(reference "R9")
+					(reference "R4")
 					(unit 1)
 				)
@@
 		(in_pos_files yes)
 		(dnp no)
-		(property "Reference" "C7"
+		(property "Reference" "C2"
 			(at 91.4463 152.4 90)
 			(show_name no)
@@
 			(project "Krteq"
 				(path "/9e7f33ad-d3b4-42c3-9373-23856f560db6"
-					(reference "C7")
+					(reference "C2")
 					(unit 1)
 				)
@@
 		(in_pos_files yes)
 		(dnp no)
-		(property "Reference" "C10"
+		(property "Reference" "C4"
 			(at 81.2863 161.29 90)
 			(show_name no)
@@
 			(project "Krteq"
 				(path "/9e7f33ad-d3b4-42c3-9373-23856f560db6"
-					(reference "C10")
+					(reference "C4")
 					(unit 1)
 				)

Commit message: BOM update
Parts:
- A1: now fitted
- C1, C2, C3, C7: footprint (none) -> Capacitor_SMD:C_01005_0402Metric; MPN (none) -> CL10B474KA8NNNC; Package (none) -> 0402
- C4, C5, C6: footprint (none) -> Capacitor_SMD:C_01005_0402Metric; MPN (none) -> CL05B104KO5NNNC; Package (none) -> 0402
- D100, D101, D102, D103, D104, D105, D106, D107, D108, D109, D110, D111, D112, D113, D114, D115, D116, D117, D118, D119, D120, D121, D122, D123, D124, D125, D65, D66, D67, D68, D69, D70, D71, D72, D73, D74, D75, D76, D77, D78, D79, D80, D81, D82, D83, D84, D85, D86, D87, D88, D89, D90, D91, D92, D93, D94, D95, D96, D97, D98, D99: MPN (none) -> A-SP1513R6GHB1C-A01-2A; Package (none) -> SMD-4P,3.2x1.3mm
- J71: now left out of the parts list
- SW1, SW10, SW11, SW12, SW13, SW14, SW15, SW16, SW17, SW18, SW19, SW2, SW20, SW21, SW22, SW23, SW24, SW25, SW26, SW27, SW28, SW29, SW3, SW30, SW32, SW33, SW34, SW35, SW36, SW37, SW38, SW39, SW4, SW40, SW41, SW42, SW43, SW44, SW45, SW46, SW47, SW48, SW49, SW5, SW50, SW51, SW52, SW53, SW54, SW55, SW56, SW57, SW58, SW59, SW6, SW60, SW61, SW7, SW8, SW9: footprint Krteq:KS-33B Hotswap 1u -> Krteq:Gateron_KS-33
- SW31: footprint Krteq:KS-33B Hotswap 2u -> Krteq:Gateron_KS-33
- U71: footprint Package_DFN_QFN:QFN-48-1EP_6x6mm_P0.4mm_EP4.2x4.2mm -> Package_DFN_QFN:QFN-48-1EP_6x6mm_P0.4mm_EP4.4x4.4mm; MPN (none) -> IS31FL3733-QFLS4-TR; Package (none) -> QFN-48-EP(6x6)
