File: source/kicad/Krteq/Krteq.kicad_sch (KiCad schematic)
At the start: 202 parts, among them J1 USB breakout board, J2 Pico test points, J3 OLED 128x32, SW1 Switch, SW10 Switch, SW11 Switch, SW12 Switch, SW13 Switch, SW14 Switch, SW15 Switch, SW16 Switch, SW17 Switch, SW18 Switch, SW19 Switch, SW2 Switch, SW20 Switch, SW21 Switch, SW22 Switch, SW23 Switch, SW24 Switch, SW25 Switch, SW26 Switch, SW27 Switch, SW28 Switch, SW29 Switch, SW3 Switch, SW30 Switch, SW31 Switch, SW32 Switch, SW33 Switch, SW34 Switch, SW35 Switch, SW36 Switch, SW37 Switch, SW38 Switch, SW39 Switch, SW4 Switch, SW40 Switch, SW41 Switch, SW42 Switch, SW43 Switch, SW44 Switch, SW45 Switch, SW46 Switch, SW47 Switch, SW48 Switch, SW49 Switch, SW5 Switch, SW50 Switch, SW51 Switch, SW52 Switch, SW53 Switch, SW54 Switch, SW55 Switch, SW56 Switch, SW57 Switch, SW58 Switch, SW59 Switch, SW6 Switch, SW60 Switch, SW61 Switch, SW7 Switch, SW8 Switch, SW9 Switch, U71 IS31FL3733-QF

Commit message: bom update
Parts:
- A1, J1, J2, J3, S1: Procurement Type (none) -> DNP; now in the parts list

Commit message: bom update
Parts:
- A1: value RaspberryPi_Pico -> Raspberry Pi Pico
- C1, C2, C3, C4: value 0.47µF -> Capacitor 0.47µF
- C5, C6, C7: value 0.1µF -> Capacitor 0.1µF
- C8: value 22µF/10V -> Capacitor 22µF/10V
- D1, D10, D11, D12, D13, D14, D15, D16, D17, D18, D19, D2, D20, D21, D22, D23, D24, D25, D26, D27, D28, D29, D3, D30, D31, D32, D33, D34, D35, D36, D37, D38, D39, D4, D40, D41, D42, D43, D44, D45, D46, D47, D48, D49, D5, D50, D51, D52, D53, D54, D55, D56, D57, D58, D59, D6, D60, D61, D7, D8, D9: value Diode -> Switch Diode
- R1, R2: value 2kΩ -> Resistor 2kΩ; MPN 0603WAF4700T5E -> 0603WAF2001T5E
- R3, R4: value 100kΩ -> Resistor 100kΩ; MPN 0603WAF4700T5E -> 0603WAF1003T5E
- R5: value 20kΩ -> Resistor 20kΩ; MPN 0603WAF4700T5E -> 0603WAF2002T5E
- SW1, SW10, SW11, SW12, SW13, SW14, SW15, SW16, SW17, SW18, SW19, SW2, SW20, SW21, SW22, SW23, SW24, SW25, SW26, SW27, SW28, SW29, SW3, SW30, SW31, SW32, SW33, SW34, SW35, SW36, SW37, SW38, SW39, SW4, SW40, SW41, SW42, SW43, SW44, SW45, SW46, SW47, SW48, SW49, SW5, SW50, SW51, SW52, SW53, SW54, SW55, SW56, SW57, SW58, SW59, SW6, SW60, SW61, SW7, SW8, SW9: value Switch -> GATERON Low Profile Switch Hot-swap Socket

Commit message: bom update
Parts:
- C1, C2, C3, C4: value Capacitor 0.47µF -> 0.47µF
- C5, C6, C7: value Capacitor 0.1µF -> 0.1µF
- C8: value Capacitor 22µF/10V -> 22µF/10V
- R1, R2: value Resistor 2kΩ -> 2kΩ
- R3, R4: value Resistor 100kΩ -> 100kΩ
- R5: value Resistor 20kΩ -> 20kΩ
Changed lines of the file:
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@@
 			)
 		)
-		(property "Value" "Resistor 20kΩ"
+		(property "Value" "20kΩ"
 			(at 63.5 207.01 90)
 			(show_name no)
@@
 			)
 		)
-		(property "Value" "Capacitor 0.47µF"
+		(property "Value" "0.47µF"
 			(at 101.6 154.178 90)
 			(show_name no)
@@
 			)
 		)
-		(property "Value" "Resistor 2kΩ"
+		(property "Value" "2kΩ"
 			(at 54.61 182.88 90)
 			(show_name no)
@@
 			)
 		)
-		(property "Value" "Resistor 100kΩ"
+		(property "Value" "100kΩ"
 			(at 48.26 203.2 90)
 			(show_name no)
@@
 			)
 		)
-		(property "Value" "Capacitor 0.1µF"
+		(property "Value" "0.1µF"
 			(at 91.44 163.068 90)
 			(show_name no)
@@
 			)
 		)
-		(property "Value" "Capacitor 0.47µF"
+		(property "Value" "0.47µF"
 			(at 63.5 173.228 90)
 			(show_name no)
@@
 			)
 		)
-		(property "Value" "Resistor 2kΩ"
+		(property "Value" "2kΩ"
 			(at 48.26 182.88 90)
 			(show_name no)
@@
 			)
 		)
-		(property "Value" "Capacitor 0.47µF"
+		(property "Value" "0.47µF"
 			(at 81.28 154.178 90)
 			(show_name no)
@@
 			)
 		)
-		(property "Value" "Resistor 100kΩ"
+		(property "Value" "100kΩ"
 			(at 54.61 204.47 90)
 			(show_name no)
@@
 			)
 		)
-		(property "Value" "Capacitor 22µF/10V"
+		(property "Value" "22µF/10V"
 			(at 69.596 154.94 0)
 			(show_name no)
@@
 			)
 		)
-		(property "Value" "Capacitor 0.1µF"
+		(property "Value" "0.1µF"
 			(at 101.6 163.068 90)
 			(show_name no)
@@
 			)
 		)
-		(property "Value" "Capacitor 0.47µF"
+		(property "Value" "0.47µF"
 			(at 91.44 154.178 90)
 			(show_name no)
@@
 			)
 		)
-		(property "Value" "Capacitor 0.1µF"
+		(property "Value" "0.1µF"
 			(at 81.28 163.068 90)
 			(show_name no)

Commit message: bom update
Parts:
- D101, D102, D103, D104, D105, D106, D107, D108, D109, D110, D111, D112, D113, D114, D115, D116, D117, D118, D119, D120, D121, D122, D123, D124, D125, D126, D127, D128, D129, D130, D131, D132, D133, D134, D135, D136, D137, D138, D139, D140, D141, D142, D143, D144, D145, D146, D147, D148, D149, D150, D151, D152, D153, D154, D155, D156, D157, D158, D159, D160, D161: value LED_ABGR -> Reverse Mount LED ABGR
- S1: value Spacebar_Stabilizer -> Spacebar Stabilizer
Changed lines of the file:
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@@
 			)
 		)
-		(property "Value" "LED_ABGR"
+		(property "Value" "Reverse Mount LED ABGR"
 			(at 184.15 208.28 0)
 			(hide yes)
@@
 			)
 		)
-		(property "Value" "LED_ABGR"
+		(property "Value" "Reverse Mount LED ABGR"
 			(at 218.44 209.55 0)
 			(hide yes)
@@
 			)
 		)
-		(property "Value" "LED_ABGR"
+		(property "Value" "Reverse Mount LED ABGR"
 			(at 218.44 189.23 0)
 			(hide yes)
@@
 			)
 		)
-		(property "Value" "LED_ABGR"
+		(property "Value" "Reverse Mount LED ABGR"
 			(at 229.87 167.64 0)
 			(hide yes)
@@
 			)
 		)
-		(property "Value" "LED_ABGR"
+		(property "Value" "Reverse Mount LED ABGR"
 			(at 275.59 208.28 0)
 			(hide yes)
@@
 			)
 		)
-		(property "Value" "LED_ABGR"
+		(property "Value" "Reverse Mount LED ABGR"
 			(at 229.87 187.96 0)
 			(hide yes)
@@
 			)
 		)
-		(property "Value" "LED_ABGR"
+		(property "Value" "Reverse Mount LED ABGR"
 			(at 298.45 167.64 0)
 			(hide yes)
@@
 			)
 		)
-		(property "Value" "LED_ABGR"
+		(property "Value" "Reverse Mount LED ABGR"
 			(at 195.58 148.59 0)
 			(hide yes)
@@
 			)
 		)
-		(property "Value" "LED_ABGR"
+		(property "Value" "Reverse Mount LED ABGR"
 			(at 264.16 209.55 0)
 			(hide yes)
@@
 			)
 		)
-		(property "Value" "LED_ABGR"
+		(property "Value" "Reverse Mount LED ABGR"
 			(at 264.16 168.91 0)
 			(hide yes)
@@
 			)
 		)
-		(property "Value" "LED_ABGR"
+		(property "Value" "Reverse Mount LED ABGR"
 			(at 321.31 187.96 0)
 			(hide yes)
@@
 			)
 		)
-		(property "Value" "LED_ABGR"
+		(property "Value" "Reverse Mount LED ABGR"
 			(at 344.17 187.96 0)
 			(hide yes)
@@
 			)
 		)
-		(property "Value" "LED_ABGR"
+		(property "Value" "Reverse Mount LED ABGR"
 			(at 207.01 187.96 0)
 			(hide yes)
@@
 			)
 		)
-		(property "Value" "LED_ABGR"
+		(property "Value" "Reverse Mount LED ABGR"
 			(at 207.01 147.32 0)
 			(hide yes)
@@
 			)
 		)
-		(property "Value" "LED_ABGR"
+		(property "Value" "Reverse Mount LED ABGR"
 			(at 275.59 187.96 0)
 			(hide yes)
@@
 			)
 		)
-		(property "Value" "LED_ABGR"
+		(property "Value" "Reverse Mount LED ABGR"
 			(at 241.3 189.23 0)
 			(hide yes)
@@
 			)
 		)
-		(property "Value" "Spacebar_Stabilizer"
+		(property "Value" "Spacebar Stabilizer"
 			(at 257.81 113.0299 0)
 			(show_name no)
@@
 			)
 		)
-		(property "Value" "LED_ABGR"
+		(property "Value" "Reverse Mount LED ABGR"
 			(at 332.74 209.55 0)
 			(hide yes)
@@
 			)
 		)
-		(property "Value" "LED_ABGR"
+		(property "Value" "Reverse Mount LED ABGR"
 			(at 321.31 147.32 0)
 			(hide yes)
@@
 			)
 		)
-		(property "Value" "LED_ABGR"
+		(property "Value" "Reverse Mount LED ABGR"
 			(at 252.73 208.28 0)
 			(hide yes)
@@
 			)
 		)
-		(property "Value" "LED_ABGR"
+		(property "Value" "Reverse Mount LED ABGR"
 			(at 207.01 167.64 0)
 			(hide yes)
@@
 			)
 		)
-		(property "Value" "LED_ABGR"
+		(property "Value" "Reverse Mount LED ABGR"
 			(at 298.45 147.32 0)
 			(hide yes)
@@
 			)
 		)
-		(property "Value" "LED_ABGR"
+		(property "Value" "Reverse Mount LED ABGR"
 			(at 309.88 148.59 0)
 			(hide yes)
@@
 			)
 		)
-		(property "Value" "LED_ABGR"
+		(property "Value" "Reverse Mount LED ABGR"
 			(at 252.73 167.64 0)
 			(hide yes)
@@
 			)
 		)
-		(property "Value" "LED_ABGR"
+		(property "Value" "Reverse Mount LED ABGR"
 			(at 287.02 168.91 0)
 			(hide yes)
@@
 			)
 		)
-		(property "Value" "LED_ABGR"
+		(property "Value" "Reverse Mount LED ABGR"
 			(at 229.87 208.28 0)
 			(hide yes)
@@
 			)
 		)
-		(property "Value" "LED_ABGR"
+		(property "Value" "Reverse Mount LED ABGR"
 			(at 241.3 209.55 0)
 			(hide yes)
@@
 			)
 		)
-		(property "Value" "LED_ABGR"
+		(property "Value" "Reverse Mount LED ABGR"
 			(at 287.02 209.55 0)
 			(hide yes)
@@
 			)
 		)
-		(property "Value" "LED_ABGR"
+		(property "Value" "Reverse Mount LED ABGR"
 			(at 252.73 187.96 0)
 			(hide yes)
@@
 			)
 		)
-		(property "Value" "LED_ABGR"
+		(property "Value" "Reverse Mount LED ABGR"
 			(at 252.73 147.32 0)
 			(hide yes)
@@
 			)
 		)
-		(property "Value" "LED_ABGR"
+		(property "Value" "Reverse Mount LED ABGR"
 			(at 241.3 148.59 0)
 			(hide yes)
@@
 			)
 		)
-		(property "Value" "LED_ABGR"
+		(property "Value" "Reverse Mount LED ABGR"
 			(at 229.87 147.32 0)
 			(hide yes)
@@
 			)
 		)
-		(property "Value" "LED_ABGR"
+		(property "Value" "Reverse Mount LED ABGR"
 			(at 321.31 208.28 0)
 			(hide yes)
@@
 			)
 		)
-		(property "Value" "LED_ABGR"
+		(property "Value" "Reverse Mount LED ABGR"
 			(at 184.15 187.96 0)
 			(hide yes)
@@
 			)
 		)
-		(property "Value" "LED_ABGR"
+		(property "Value" "Reverse Mount LED ABGR"
 			(at 195.58 168.91 0)
 			(hide yes)
@@
 			)
 		)
-		(property "Value" "LED_ABGR"
+		(property "Value" "Reverse Mount LED ABGR"
 			(at 344.17 147.32 0)
 			(hide yes)
@@
 			)
 		)
-		(property "Value" "LED_ABGR"
+		(property "Value" "Reverse Mount LED ABGR"
 			(at 218.44 168.91 0)
 			(hide yes)
@@
 			)
 		)
-		(property "Value" "LED_ABGR"
+		(property "Value" "Reverse Mount LED ABGR"
 			(at 264.16 148.59 0)
 			(hide yes)
@@
 			)
 		)
-		(property "Value" "LED_ABGR"
+		(property "Value" "Reverse Mount LED ABGR"
 			(at 321.31 167.64 0)
 			(hide yes)
@@
 			)
 		)
-		(property "Value" "LED_ABGR"
+		(property "Value" "Reverse Mount LED ABGR"
 			(at 298.45 208.28 0)
 			(hide yes)
@@
 			)
 		)
-		(property "Value" "LED_ABGR"
+		(property "Value" "Reverse Mount LED ABGR"
 			(at 195.58 209.55 0)
 			(hide yes)
@@
 			)
 		)
-		(property "Value" "LED_ABGR"
+		(property "Value" "Reverse Mount LED ABGR"
 			(at 172.72 148.59 0)
 			(hide yes)
@@
 			)
 		)
-		(property "Value" "LED_ABGR"
+		(property "Value" "Reverse Mount LED ABGR"
 			(at 344.17 208.28 0)
 			(hide yes)
@@
 			)
 		)
-		(property "Value" "LED_ABGR"
+		(property "Value" "Reverse Mount LED ABGR"
 			(at 287.02 189.23 0)
 			(hide yes)
@@
 			)
 		)
-		(property "Value" "LED_ABGR"
+		(property "Value" "Reverse Mount LED ABGR"
 			(at 195.58 189.23 0)
 			(hide yes)
@@
 			)
 		)
-		(property "Value" "LED_ABGR"
+		(property "Value" "Reverse Mount LED ABGR"
 			(at 332.74 189.23 0)
 			(hide yes)
@@
 			)
 		)
-		(property "Value" "LED_ABGR"
+		(property "Value" "Reverse Mount LED ABGR"
 			(at 184.15 167.64 0)
 			(hide yes)
@@
 			)
 		)
-		(property "Value" "LED_ABGR"
+		(property "Value" "Reverse Mount LED ABGR"
 			(at 344.17 167.64 0)
 			(hide yes)
@@
 			)
 		)
-		(property "Value" "LED_ABGR"
+		(property "Value" "Reverse Mount LED ABGR"
 			(at 287.02 148.59 0)
 			(hide yes)
@@
 			)
 		)
-		(property "Value" "LED_ABGR"
+		(property "Value" "Reverse Mount LED ABGR"
 			(at 241.3 168.91 0)
 			(hide yes)
@@
 			)
 		)
-		(property "Value" "LED_ABGR"
+		(property "Value" "Reverse Mount LED ABGR"
 			(at 264.16 189.23 0)
 			(hide yes)
@@
 			)
 		)
-		(property "Value" "LED_ABGR"
+		(property "Value" "Reverse Mount LED ABGR"
 			(at 172.72 209.55 0)
 			(hide yes)
@@
 			)
 		)
-		(property "Value" "LED_ABGR"
+		(property "Value" "Reverse Mount LED ABGR"
 			(at 207.01 208.28 0)
 			(hide yes)
@@
 			)
 		)
-		(property "Value" "LED_ABGR"
+		(property "Value" "Reverse Mount LED ABGR"
 			(at 309.88 189.23 0)
 			(hide yes)
@@
 			)
 		)
-		(property "Value" "LED_ABGR"
+		(property "Value" "Reverse Mount LED ABGR"
 			(at 298.45 187.96 0)
 			(hide yes)
@@
 			)
 		)
-		(property "Value" "LED_ABGR"
+		(property "Value" "Reverse Mount LED ABGR"
 			(at 275.59 147.32 0)
 			(hide yes)
@@
 			)
 		)
-		(property "Value" "LED_ABGR"
+		(property "Value" "Reverse Mount LED ABGR"
 			(at 309.88 209.55 0)
 			(hide yes)
@@
 			)
 		)
-		(property "Value" "LED_ABGR"
+		(property "Value" "Reverse Mount LED ABGR"
 			(at 218.44 148.59 0)
 			(hide yes)
@@
 			)
 		)
-		(property "Value" "LED_ABGR"
+		(property "Value" "Reverse Mount LED ABGR"
 			(at 309.88 168.91 0)
 			(hide yes)
@@
 			)
 		)
-		(property "Value" "LED_ABGR"
+		(property "Value" "Reverse Mount LED ABGR"
 			(at 184.15 147.32 0)
 			(hide yes)
@@
 			)
 		)
-		(property "Value" "LED_ABGR"
+		(property "Value" "Reverse Mount LED ABGR"
 			(at 332.74 148.59 0)
 			(hide yes)
@@
 			)
 		)
-		(property "Value" "LED_ABGR"
+		(property "Value" "Reverse Mount LED ABGR"
 			(at 275.59 167.64 0)
 			(hide yes)

Commit message: update
Parts:
- U71: footprint Package_DFN_QFN:QFN-48-1EP_6x6mm_P0.4mm_EP4.4x4.4mm -> Krteq:QFN-48_6x6mm
Changed lines of the file:
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@@
 			)
 		)
-		(property "Footprint" "Package_DFN_QFN:QFN-48-1EP_6x6mm_P0.4mm_EP4.4x4.4mm"
+		(property "Footprint" "Krteq:QFN-48_6x6mm"
 			(at 86.36 219.71 0)
 			(hide yes)

Commit message: update
Parts:
- U71: value IS31FL3733-QF -> LED Driver
Changed lines of the file:
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@@
 			)
 		)
-		(property "Value" "IS31FL3733-QF"
+		(property "Value" "LED Driver"
 			(at 91.0433 262.89 0)
 			(show_name no)

Commit message: update
Connections:
- net 3V3: now also J3.3 (Pin_3); no longer J3.1 (Pin_1)
- net DATA+: now also J1.4 (Pin_4), J2.3 (Pin_3); no longer J1.3 (Pin_3), J2.2 (Pin_2)
- net DATA-: now also J1.3 (Pin_3); no longer J1.4 (Pin_4)
- net GND: now also J1.1 (Pin_1), J2.2 (Pin_2); no longer J1.2 (Pin_2), J2.3 (Pin_3)
- net SCL: now also J3.2 (Pin_2); no longer J3.3 (Pin_3)
- net SDA: now also J3.1 (Pin_1); no longer J3.2 (Pin_2)
- net VBUS: now also J1.2 (Pin_2); no longer J1.1 (Pin_1)

Commit message: better capacitor
Parts:
- C8: footprint Capacitor_SMD:C_0805_2012Metric -> Krteq:CASE-A-3216-18(mm); symbol Device:C_Small -> Device:C_Polarized_Small
Changed lines of the file:
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@@
 	)
 	(symbol
-		(lib_id "Device:C_Small")
+		(lib_id "Device:C_Polarized_Small")
 		(at 72.39 153.67 0)
 		(unit 1)
@@
 			)
 		)
-		(property "Footprint" "Capacitor_SMD:C_0805_2012Metric"
+		(property "Footprint" "Krteq:CASE-A-3216-18(mm)"
 			(at 72.39 153.67 0)
 			(hide yes)
@@
 			)
 		)
-		(property "Description" "Unpolarized capacitor, small symbol"
+		(property "Description" "Polarized capacitor, small symbol"
 			(at 72.39 153.67 0)
 			(hide yes)
