File: source/kicad/Krteq/Krteq.kicad_pcb (KiCad board)
At the start: 2 copper layers, 228.6 x 114.3 mm, 199 parts, among them J71 OLED 128x32, SW1 Switch, SW10 Switch, SW11 Switch, SW12 Switch, SW13 Switch, SW14 Switch, SW15 Switch, SW16 Switch, SW17 Switch, SW18 Switch, SW19 Switch, SW2 Switch, SW20 Switch, SW21 Switch, SW22 Switch, SW23 Switch, SW24 Switch, SW25 Switch, SW26 Switch, SW27 Switch, SW28 Switch, SW29 Switch, SW3 Switch, SW30 Switch, SW31 Switch, SW32 Switch, SW33 Switch, SW34 Switch, SW35 Switch, SW36 Switch, SW37 Switch, SW38 Switch, SW39 Switch, SW4 Switch, SW40 Switch, SW41 Switch, SW42 Switch, SW43 Switch, SW44 Switch, SW45 Switch, SW46 Switch, SW47 Switch, SW48 Switch, SW49 Switch, SW5 Switch, SW50 Switch, SW51 Switch, SW52 Switch, SW53 Switch, SW54 Switch, SW55 Switch, SW56 Switch, SW57 Switch, SW58 Switch, SW59 Switch, SW6 Switch, SW60 Switch, SW61 Switch, SW7 Switch, SW8 Switch, SW9 Switch, U71 IS31FL3733-QF

Commit message: update
Parts:
- A1: moved to F.Cu
- turned A1 to -90 degrees

Commit message: update
Parts:
- removed J71: OLED 128x32, Krteq:Display_Module
- added J1: Pico test points, Krteq:Interface_1x04_P2.54mm, B.Cu at (192.9, 86.9)
- added J2: USB breakout board, Krteq:Interface_1x04_P2.54mm, B.Cu at (292.4, 86.9)
- added J3: OLED 128x32, Krteq:Interface_1x04_P2.54mm, B.Cu at (245.9, 86.9)
- moved A1 110.2 mm to (156.4, 87.8)
- moved U71 85.0 mm to (263.0, 86.3)
- moved C1 80.6 mm to (273.6, 84.9)
- moved C2 80.6 mm to (276.6, 79.9)
- moved C3 80.6 mm to (273.6, 79.9)
- moved C4 80.6 mm to (270.6, 79.9)
- moved C5 80.6 mm to (276.6, 81.9)
- moved C6 80.6 mm to (273.6, 81.9)
- moved C7 80.6 mm to (270.6, 81.9)
- moved R1 80.6 mm to (277.6, 84.9)
- moved R2 80.6 mm to (277.6, 86.9)
- moved R3 80.6 mm to (277.6, 88.9)
- moved R4 80.6 mm to (277.6, 90.9)
- moved R5 80.6 mm to (277.6, 92.9)
Other:
- outline, holes or cut-outs redrawn

Commit message: update
Parts:
- A1: moved to B.Cu
- turned A1 to 90 degrees
Other:
- outline, holes or cut-outs redrawn

Commit message: update
Parts:
- J1: value Pico test points -> USB breakout board
- J2: value USB breakout board -> Pico test points; footprint Krteq:Interface_1x04_P2.54mm -> Krteq:Interface_1x03_P2.54mm
- moved J1 99.8 mm to (292.4, 79.4), turned to 180 degrees
- moved J2 99.3 mm to (193.4, 79.4), turned to 180 degrees
- moved D2 8.58 mm to (311.4, 90.9), turned to 0 degrees
- moved J3 7.54 mm to (245.9, 79.4), turned to 180 degrees
Connections:
- A1 pad 1: unconnected-(A1-GPIO0-Pad1) -> SDA
- A1 pad 10: unconnected-(A1-GPIO7-Pad10) -> COL7
- A1 pad 11: unconnected-(A1-GPIO8-Pad11) -> COL6
- A1 pad 12: unconnected-(A1-GPIO9-Pad12) -> COL5
- A1 pad 14: unconnected-(A1-GPIO10-Pad14) -> COL4
- A1 pad 15: unconnected-(A1-GPIO11-Pad15) -> COL3
- A1 pad 16: unconnected-(A1-GPIO12-Pad16) -> COL2
- A1 pad 17: SDB -> unconnected-(A1-GPIO13-Pad17)
- A1 pad 19: SDA -> unconnected-(A1-GPIO14-Pad19)
- A1 pad 2: unconnected-(A1-GPIO1-Pad2) -> SCL
- A1 pad 20: SCL -> COL0
- A1 pad 21: unconnected-(A1-GPIO16-Pad21) -> ROW0
- A1 pad 22: unconnected-(A1-GPIO17-Pad22) -> ROW1
- A1 pad 24: unconnected-(A1-GPIO18-Pad24) -> COL1
- A1 pad 25: unconnected-(A1-GPIO19-Pad25) -> ROW2
- A1 pad 26: unconnected-(A1-GPIO20-Pad26) -> ROW3
- A1 pad 27: unconnected-(A1-GPIO21-Pad27) -> ROW4
- A1 pad 29: unconnected-(A1-GPIO22-Pad29) -> ROW5
- A1 pad 4: unconnected-(A1-GPIO2-Pad4) -> SDB
- A1 pad 5: unconnected-(A1-GPIO3-Pad5) -> COL11
- A1 pad 6: unconnected-(A1-GPIO4-Pad6) -> COL10
- A1 pad 7: unconnected-(A1-GPIO5-Pad7) -> COL9
- A1 pad 9: unconnected-(A1-GPIO6-Pad9) -> COL8
- J1 pad 1: USB GND -> GND
- J1 pad 2: USB D+ -> DATA+
- J1 pad 3: USB D- -> DATA-
- J1 pad 4: USB VBUS -> VBUS
- J2 pad 1: USB GND -> GND
- J2 pad 2: USB D+ -> DATA-
- J2 pad 3: USB D- -> DATA+

Commit message: update
Parts:
- moved J3 0.68 mm to (245.5, 78.9)
- moved J1 0.59 mm to (292.7, 78.9)
- moved J2 0.55 mm to (193.5, 78.9)
Changed lines of the file:
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@@
 		(capping no)
 		(filling no)
-		(grid_origin 219.425 95.925)
+		(grid_origin 294.725 76.875)
 		(pcbplotparams
 			(layerselection 0x00000000_00000000_55555555_5755f5ff)
@@
 	(footprint "Krteq:Interface_1x03_P2.54mm"
 		(layer "B.Cu")
-		(at 193.425 79.425 180)
+		(at 193.475 78.875 180)
 		(descr "Through hole straight pin header, 1x04, 2.54mm pitch, single row")
 		(tags "Through hole pin header THT 1x04 2.54mm single row")
@@
 	(footprint "Krteq:Interface_1x04_P2.54mm"
 		(layer "B.Cu")
-		(at 245.925 79.385 180)
+		(at 245.475 78.875 180)
 		(descr "Through hole straight pin header, 1x04, 2.54mm pitch, single row")
 		(tags "Through hole pin header THT 1x04 2.54mm single row")
@@
 	(footprint "Krteq:Interface_1x04_P2.54mm"
 		(layer "B.Cu")
-		(at 292.425 79.385 180)
+		(at 292.725 78.875 180)
 		(descr "Through hole straight pin header, 1x04, 2.54mm pitch, single row")
 		(tags "Through hole pin header THT 1x04 2.54mm single row")

Commit message: update
Connections:
- J3 pad 2: 3V3 -> SDA
- J3 pad 4: SDA -> 3V3
Changed lines of the file:
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@@
 		(descr "Through hole straight pin header, 1x04, 2.54mm pitch, single row")
 		(tags "Through hole pin header THT 1x04 2.54mm single row")
+		(property "Reference" "J2"
+			(at 0 -7.62 0)
+			(layer "B.SilkS")
+			(effects
+				(font
+					(size 1 1)
+					(thickness 0.15)
+				)
+				(justify mirror)
+			)
+		)
 		(property "Value" "Pico test points"
 			(at 0 2.54 0)
@@
 			)
 		)
-		(property "Description" "Generic connector, single row, 01x03, script generated"
+		(property "Description" "Generic connector, single row, 01x03"
 			(at 0 0 0)
 			(layer "B.Fab")
@@
 			)
 		)
-		(property "Reference" "J2"
-			(at 0 -7.62 0)
+		(property "KiLib_Generator" "connector/pin_header_socket"
+			(at 0 0 0)
 			(layer "B.SilkS")
+			(hide yes)
 			(effects
 				(font
@@
 		(sheetname "/")
 		(sheetfile "Krteq.kicad_sch")
-		(units
-			(unit
-				(name "A")
-				(pins "1" "2" "3")
-			)
-		)
-		(attr through_hole)
+		(attr through_hole exclude_from_bom)
 		(duplicate_pad_numbers_are_jumpers no)
 		(fp_rect
-			(start -1.27 1.5)
-			(end 1.27 -6.5)
+			(start -1.25 1.25)
+			(end 1.25 -6.33)
 			(stroke
 				(width 0.05)
@@
 		(descr "Through hole straight pin header, 1x04, 2.54mm pitch, single row")
 		(tags "Through hole pin header THT 1x04 2.54mm single row")
+		(property "Reference" "J3"
+			(at 0 -10.16 0)
+			(layer "B.SilkS")
+			(effects
+				(font
+					(size 1 1)
+					(thickness 0.15)
+				)
+				(justify mirror)
+			)
+		)
 		(property "Value" "OLED 128x32"
 			(at 0 2.54 0)
@@
 			)
 		)
-		(property "Description" "Generic connector, single row, 01x04, script generated"
+		(property "Description" "Generic connector, single row, 01x04"
 			(at 0 0 0)
 			(layer "B.Fab")
@@
 			)
 		)
-		(property "Reference" "J3"
-			(at 0 -10.16 0)
+		(property "KiLib_Generator" "connector/pin_header_socket"
+			(at 0 0 0)
 			(layer "B.SilkS")
+			(hide yes)
 			(effects
 				(font
@@
 		(sheetname "/")
 		(sheetfile "Krteq.kicad_sch")
-		(units
-			(unit
-				(name "A")
-				(pins "1" "2" "3" "4")
-			)
-		)
 		(attr through_hole exclude_from_bom)
 		(duplicate_pad_numbers_are_jumpers no)
 		(fp_rect
-			(start -1.27 1.5)
-			(end 1.27 -9)
+			(start -1.25 1.25)
+			(end 1.25 -8.87)
 			(stroke
 				(width 0.05)
@@
 			(layers "*.Cu" "*.Mask")
 			(remove_unused_layers no)
-			(net "3V3")
+			(net "SDA")
 			(pinfunction "Pin_2_2")
 			(pintype "passive")
@@
 			(layers "*.Cu" "*.Mask")
 			(remove_unused_layers no)
-			(net "SDA")
+			(net "3V3")
 			(pinfunction "Pin_4_4")
 			(pintype "passive")
@@
 			)
 		)
-		(property "Description" "Generic connector, single row, 01x04, script generated"
+		(property "Description" "Generic connector, single row, 01x04"
 			(at 0 0 0)
 			(layer "B.Fab")
@@
 			)
 		)
+		(property "KiLib_Generator" "connector/pin_header_socket"
+			(at 0 0 0)
+			(layer "B.SilkS")
+			(hide yes)
+			(effects
+				(font
+					(size 1 1)
+					(thickness 0.15)
+				)
+				(justify mirror)
+			)
+		)
 		(property ki_fp_filters "Connector*:*_1x??_*")
 		(sheetname "/")
 		(sheetfile "Krteq.kicad_sch")
-		(units
-			(unit
-				(name "A")
-				(pins "1" "2" "3" "4")
-			)
-		)
 		(attr through_hole exclude_from_bom)
 		(duplicate_pad_numbers_are_jumpers no)
 		(fp_rect
-			(start -1.27 1.5)
-			(end 1.27 -9)
+			(start -1.25 1.25)
+			(end 1.25 -8.87)
 			(stroke
 				(width 0.05)
